File: bowelProbe.kicad_sch (KiCad schematic)
At the start: 52 parts, among them J10 Conn_01x01, J11 Conn_01x01, J12 Conn_01x01, J13 Conn_01x01, J2 Conn_01x01, J3 Conn_01x01, J4 Conn_01x01, J5 Conn_01x01, J6 Conn_01x01, J7 Conn_01x01, J8 Conn_01x01, J9 Conn_01x01, U1 MAX038CPP, U2 OPA2134PA, U3 MCP6002-E/P, U4 TL072ACP

Commit message: Finished Electronic Schematic, Awaiting Finalizations and Review
Added many symbols, footprints, and 3d models. Organized design into functional blocks.

Still need finalized plans and footprints for "demo".

Next Steps:
 - Finalize "demo" subciruit
 - Review schematic

- Move on to layout

- Make code for full device operation
Parts:
- removed A1: Arduino_Nano_v2.x, Module:Arduino_Nano, symbol MCU_Module:Arduino_Nano_v2.x
- removed C1, C2, C3, C4: 10u, BowelProbe:Capacitor-10u, symbol Device:C_Polarized_Small_US
- removed C7: 1n, BowelProbe:Capacitor-10n, symbol Device:C_Small
- removed D1, D2, D3: 1N5817, BowelProbe:1N5817, symbol Diode:1N4001
- removed J12, J13, J3, J4, J6, J8: Conn_01x01, BowelProbe:CT3149-0, symbol Connector_Generic:Conn_01x01
- removed J5, J7, J9: Conn_01x01, BowelProbe:CT3149-2, symbol Connector_Generic:Conn_01x01
- removed R8: 20k, BowelProbe:Resistor-20k, symbol Device:R_US
- removed U1: MAX038CPP, BowelProbe:MAX038CPP, symbol BowelProbe:MAX038CPP
- removed U2: OPA2134PA, BowelProbe:DIP794W45P254L959H508Q8, symbol OPA2134PA:OPA2134PA
- removed U3: MCP6002-E/P, BowelProbe:PDIP8_300MC_MCH, symbol MCP6002-E/P:MCP6002-E_P
- removed U4: TL072ACP, BowelProbe:P8, symbol TL072ACP:TL072ACP
- added C1, C18, C19, C20, C25, C26, C29, C30, C32, C34, C39, C40: 0.1u, BowelProbe:Cap0.1uF, symbol Device:C_Small
- added C2, C21, C24, C27, C28, C31, C33: 10u, BowelProbe:Cap10uF, symbol Device:C_Small
- added C22: 2.2n, BowelProbe:Cap2.2nF, symbol Device:C_Small
- added C23: 1n, BowelProbe:Cap1nF, symbol Device:C_Small
- added C3: 1u, BowelProbe:Cap1uF, symbol Device:C_Small
- added C35, C36: 1u, BowelProbe:Cap0.1uF, symbol Device:C_Small
- added C37, C38: 18p, BowelProbe:Cap18pF, symbol Device:C_Small
- added C4, C7: 4.7u, BowelProbe:Cap4.7uF, symbol BowelProbe:Cap4.7uF
- added CR1, CR2: DiodeClamper, BowelProbe:DiodeClamper, symbol BowelProbe:DiodeClamper
- added D1, D3: SchottkyDiode, BowelProbe:SchottkyDiode, symbol BowelProbe:SchottkyDiode
- added D2: LED_Small, symbol Device:LED_Small
- added HS1: Heatsink, BowelProbe:Heatsink, symbol BowelProbe:Heatsink
- added J1: Conn_01x01, BowelProbe:CT3149-0, symbol Connector_Generic:Conn_01x01
- added J5: Conn_02x03_Odd_Even, symbol Connector_Generic:Conn_02x03_Odd_Even
- added J6: Conn_01x08, symbol Connector_Generic:Conn_01x08
- added L1: LPD5030-472MRC, BowelProbe:InductorCoupled, symbol BowelProbe:InductorCoupled
- added L2: 10u, BowelProbe:Inductor10uH, symbol Device:L_Small
- added LS1: Speaker, symbol Device:Speaker
- added R13: 10k, BowelProbe:Resistor10k, symbol Device:R_US
- added U1: L7805CV, BowelProbe:L7805CV, symbol BowelProbe:L7805CV
- added U2: LT8330, BowelProbe:LT8330, symbol BowelProbe:LT8330
- added U3: AD9833BRMZ, BowelProbe:AD9833, symbol BowelProbe:AD9833BRMZ
- added U4: OPA2134UA/2K5, BowelProbe:OPA2134smd, symbol BowelProbe:OPA2134smd
- added U5: TL072smd, BowelProbe:TL072smd, symbol BowelProbe:TL072smd
- added U6: DiodeLowLeak, BowelProbe:DiodeLowLeak, symbol BowelProbe:DiodeLowLeak
- added U7: MCP6002-E/MC, BowelProbe:MCP6002smd, symbol BowelProbe:MCP6002smd
- added U8: ATmega328P, BowelProbe:ATmega328P, symbol BowelProbe:ATmega328P
- added XTAL1: TSX-3225 16.0000MF09Z-AC3, BowelProbe:Crystal16MHz, symbol BowelProbe:Crystal16MHz
- C10, C14, C8: value 1u -> 10u; footprint BowelProbe:Capacitor-10n -> BowelProbe:Cap10uF; Order https://www.digikey.com/en/products/detail/kemet/C330C105M5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 -> (none)
- C11, C12, C13, C15, C16, C17: value 0.1u -> 10u; footprint BowelProbe:Capacitor-10n -> BowelProbe:Cap10uF; Order https://www.digikey.com/en/products/detail/kemet/C320C104K5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 -> (none)
- C5: value 10n -> 1u; footprint BowelProbe:Capacitor-10n -> BowelProbe:Cap1uF; Order https://www.digikey.com/en/products/detail/kemet/C322C103J5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 -> (none)
- C6: value 10n -> 4.7p; footprint BowelProbe:Capacitor-10n -> BowelProbe:Cap4.7pF; Order https://www.digikey.com/en/products/detail/kemet/C322C103J5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 -> (none)
- C9: value 1n -> 10u; footprint BowelProbe:Capacitor-10n -> BowelProbe:Cap10uF; Order https://www.digikey.com/en/products/detail/kemet/C315C102M1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 -> (none)
- R1, R12, R3: value 20k -> 10k; footprint BowelProbe:Resistor-20k -> BowelProbe:Resistor10k; Order https://www.digikey.com/en/products/detail/yageo/MFR-25FRF5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 -> (none)
- R10: value 10k -> 1k; footprint BowelProbe:Resistor-20k -> BowelProbe:Resistor1k; Order https://www.digikey.com/en/products/detail/yageo/MFR-25FRF5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 -> (none)
- R11: value 20k -> 1k; footprint BowelProbe:Resistor-20k -> BowelProbe:Resistor1k; Order https://www.digikey.com/en/products/detail/yageo/MFR-25FRF5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 -> (none)
- R14: value 300k -> 10k; footprint BowelProbe:Resistor-20k -> BowelProbe:Resistor10k; Order https://www.digikey.com/en/products/detail/yageo/MFR-25FTF5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 -> (none)
- R15: value 1k -> 100; footprint BowelProbe:Resistor-20k -> BowelProbe:Resistor100; Order https://www.digikey.com/en/products/detail/yageo/MFR-25FRF5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 -> (none)
- R2: value 20k -> 1M; footprint BowelProbe:Resistor-20k -> BowelProbe:Resistor1M; Order https://www.digikey.com/en/products/detail/yageo/MFR-25FRF5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 -> (none)
- R4: value 20k -> 6.8k; footprint BowelProbe:Resistor-20k -> BowelProbe:Resistor6.8k; Order https://www.digikey.com/en/products/detail/yageo/MFR-25FRF5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 -> (none)
- R5: value 10k -> 6.8k; footprint BowelProbe:Resistor-20k -> BowelProbe:Resistor6.8k; Order https://www.digikey.com/en/products/detail/yageo/MFR-25FRF5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 -> (none)
- R6: value 10k -> 30k; footprint BowelProbe:Resistor-20k -> BowelProbe:Resistor30k; Order https://www.digikey.com/en/products/detail/yageo/MFR-25FRF5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 -> (none)
- R7: value 10k -> 1.8k; footprint BowelProbe:Resistor-20k -> BowelProbe:Resistor1.8k; Order https://www.digikey.com/en/products/detail/yageo/MFR-25FRF5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 -> (none)
- R8: renamed from R13; footprint BowelProbe:Resistor-20k -> BowelProbe:Resistor100; Order https://www.digikey.com/en/products/detail/yageo/MFR100FTF5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 -> (none)
- R9: value 25k -> 300k; footprint BowelProbe:Resistor-20k -> BowelProbe:Resistor300k; Order https://www.digikey.com/en/products/detail/vishay-dale/RN60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 -> (none)
- renumbered J10 to J3, J11 to J4
Connections:
- net GND: now also C11.2, C12.2, C13.2, C14.2, C16.2, C8.2, R1.2, R11.2, R15.2, R9.2, C1.2, C18.2, C2.2, C20.1, C23.1, C24.2, C25.2, C26.1, C27.1, C28.2, C29.2, C3.2, C30.1, C31.1, C32.2, C33.2, C34.2, C35.2, C36.2, C37.1, C38.1, C39.2, C4.1, C40.2, C7.1, CR1.1, CR2.2, D1.C, HS1.1, HS1.2, J1.1 (Pin_1), J5.6 (Pin_6), J6.3 (Pin_3), U1.2 (GROUND), U2.5 (GND), U2.9 (GND), U3.4 (DGND), U3.9 (AGND), U4.5 (INB+), U7.4 (VSS), U7.9 (EPAD), U8.21 (GND), U8.3 (GND), U8.33 (GND), U8.5 (GND), XTAL1.2, XTAL1.4; no longer C11.1, C12.1, C13.1, C14.1, C16.1, C5.1, C6.1, C8.1, R10.1, R14.2
- net at R1.1: now also C6.2, R2.1, U2.1 (FBX); no longer R5.1
- net +12V: now reaches J2.1 (Pin_1)
- net +12V: now also C10.1, C8.1, C9.1, C1.1, C26.2, C27.2, C30.2, C31.2, C4.2, L1.1, U1.1 (INPUT), U2.6 (VIN), U2.8 (EN/UVLO), U4.8 (V+), U5.8 (VCC+); no longer C8.2
- net -12V: now reaches C15.1
- net -12V: now also C14.1, C16.1, C6.1, R2.2, C24.1, C25.1, C28.1, C29.1, C7.2, L1.4, U4.4 (V-), U5.4 (VCC-); no longer C12.2
- net Vfiltered: now reaches R7.2
- net Vfiltered: now also C22.1, U4.1 (OUTA), U4.2 (INA-); no longer R4.1
- net Vprobe: now reaches J3.1 (Pin_1), R8.2
- net Vprobe: now also U5.3 (1IN+)
- net at R6.2, R7.1: now also U4.6 (INB-); no longer R3.1
- net nReset: now reaches R12.1
- net nReset: now also J5.5 (Pin_5), U8.29 (PC6)
- net VADCbuf: now reaches R10.2
- net VADCbuf: now also CR1.2, CR2.1, U7.5 (VINB+); no longer R11.2
- net Vamplified: now reaches R8.1
- net Vamplified: now also R6.1, U4.7 (OUTB)
- net at R11.1: now also D2.1 (K); no longer R12.2
- net at R9.1: now also R10.1, C32.1, U5.6 (2IN-), U6.3
- net +5V: now reaches R3.2
- net +5V: now also C11.1, C12.1, C13.1, C17.1, R12.2, R14.2, C18.1, C19.2, C2.1, C33.1, C34.1, C35.1, C36.1, J5.2 (Pin_2), J6.1 (Pin_1), L2.2, R13.2, U1.3 (OUTPUT), U3.2 (VDD), U7.8 (VDD), U8.4 (VCC), U8.6 (VCC)
- net at C5.2: now also L1.2, U2.3 (SW), U2.4 (SW); no longer C6.2
- net at R4.2: now also R5.1, C22.2
- new net: C21.1, U3.10 (VOUT)
- new net: U5.7 (2OUT), U6.1
- new net: C19.1, U3.1 (COMP)
- new net: C38.2, U8.8 (PB7), XTAL1.3
- new net: D3.A, LS1.2, R15.1
- new net: C3.1, U2.7 (INTVCC)
- new net: C40.1, L2.1, U8.18 (AVCC)
- new net: C20.2, U3.3 (CAP/2.5V)
- new net: C5.1, D1.A, L1.3
- new net: C39.1, U8.20 (AREF)
- new net: C37.2, U8.7 (PB6), XTAL1.1
- new net: C23.2, R5.2, U4.3 (INA+)
- new net CD: J6.8 (Pin_8), R14.1, U8.13 (PB1)
- new net CLKO: U3.5 (MCLK), U8.12 (PB0)
- new net MISO: J5.1 (Pin_1), J6.5 (Pin_5), U8.16 (PB4)
- new net MOSI: J5.4 (Pin_4), J6.6 (Pin_6), U3.6 (SDATA), U8.15 (PB3)
- new net SCK: J5.3 (Pin_3), J6.4 (Pin_4), U3.7 (SCLK), U8.17 (PB5)
- new net Test1: D2.2 (A), U8.32 (PD2)
- new net Test2: D3.C, LS1.1, U8.10 (PD6)
- new net VADC: U7.6 (VINB-), U7.7 (VOUTB), U8.23 (PC0)
- new net Vbuffer: U5.1 (1OUT), U5.2 (1IN-), U5.5 (2IN+)
- new net Vsingen: C21.2, R4.1
- new net nSS: J6.7 (Pin_7), R13.1, U8.14 (PB2)
- new net nSS_Sin: R3.1, U3.8 (FSYNC), U8.25 (PC2)
- no-connect marks 25 -> 5
Other:
- note added: "ADC"
- note added: "ATmega328P & Demo"
- note added: "Buffer & Superdiode Peak Detector"
- note added: "ICSP"
- note added: "Long Power Trace Decoupling"
- note added: "MicroSD"
- note added: "Pin 1 - 5V Pin 2 - 3V Pin 3 - GND Pin 4 - CLK Pin 5 - DO Pin 6 - DI Pin 7 - CS Pin 8 - CD"
- note added: "Pin 1 - D12 Pin 2 - Vcc Pin 3 - D13 Pin 4 - D11 Pin 5 - D10 Pin 6 - GND"
- note added: "Power"
- note added: "Sine Amplification"
- note added: "Sine Generation"
- note added: "Voltage Divider"
- note removed: "(LSB)"
- note removed: "(MSB)"
- note removed: "+12V"
- note removed: "+5V"
- note removed: "-12V"
- note removed: "-5V"
- moved on the sheet: R8

Commit message: Schematic Finalized and Reviewed, Awaiting Professor Review
Schematic finalized, corrected, and finished. Awaiting professor review.

Next steps:
- PCB layout
- Programming
- Update BOM
Parts:
- removed D2: LED_Small, symbol Device:LED_Small
- removed D3: SchottkyDiode, BowelProbe:SchottkyDiode, symbol BowelProbe:SchottkyDiode
- removed LS1: Speaker, symbol Device:Speaker
- removed R11: 1k, BowelProbe:Resistor1k, symbol Device:R_US
- removed R15: 100, BowelProbe:Resistor100, symbol Device:R_US
- added J10, J11, J12, J13, J14, J15, J16, J17, J18, J19, J20, J7, J8, J9: Conn_01x01, BowelProbe:CT3149-0, symbol Connector_Generic:Conn_01x01
- J5: footprint (none) -> BowelProbe:Dupont2x3
- J6: footprint (none) -> BowelProbe:microSD
- R1: value 10k -> 71.5k; footprint BowelProbe:Resistor10k -> BowelProbe:Resistor71.5k
- U5: value TL072smd -> TL072ACDR
Connections:
- net +5V: now also CR1.1
- net GND: now also R8.2; no longer CR1.1, J4.1 (Pin_1)
- net VADC: now also U8.22 (ADC7); no longer U8.23 (PC0)
- net Vamplified: now also J3.1 (Pin_1); no longer R8.1
- net Vprobe: now also J4.1 (Pin_1), R8.1; no longer J3.1 (Pin_1), R8.2
- net D3: now reaches U8.1 (PD3)
- net D3: now also J10.1 (Pin_1)
- net D7: now reaches U8.11 (PD7)
- net D7: now also J14.1 (Pin_1)
- net A6: now reaches U8.19 (ADC6)
- net D4: now reaches U8.2 (PD4)
- net D4: now also J11.1 (Pin_1)
- net A1: now reaches U8.24 (PC1)
- net A1: now also J16.1 (Pin_1)
- net A3: now reaches U8.26 (PC3)
- net A3: now also J18.1 (Pin_1)
- net A4: now reaches U8.27 (PC4)
- net A4: now also J19.1 (Pin_1)
- net A5: now reaches U8.28 (PC5)
- net A5: now also J20.1 (Pin_1)
- net D0: now reaches U8.30 (PD0)
- net D0: now also J7.1 (Pin_1)
- net D1: now reaches U8.31 (PD1)
- net D1: now also J8.1 (Pin_1)
- net D5: now reaches U8.9 (PD5)
- net D5: now also J12.1 (Pin_1)
- net Test1 renamed D2
- net D2: now also J9.1 (Pin_1)
- net Test2 renamed D6
- net D6: now also J13.1 (Pin_1)
- new net A0: J15.1 (Pin_1), U8.23 (PC0)
- new net A2: J17.1 (Pin_1)
Other:
- note added: "Extra Pins"
- moved on the sheet: C10, C11, C12, C13, C14, C15, C16, C39, C8, C9, J3, J4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

Commit message: LTspice Source Scripting
Created python script to model sine wave generator (replacement model for chip AD9833 w/o spice model). Additionally began initial pcb placement.
Parts:
- C1, C18, C19, C20, C25, C26, C29, C30, C32, C34, C39, C40: Manufacturer (none) -> Murata Electronics; Manufacturer Product Number (none) -> GRM033C71C104KE14D
- C10, C11, C12, C13, C14, C15, C16, C17, C2, C21, C24, C27, C28, C31, C33, C8, C9: Manufacturer (none) -> Murata Electronics; Manufacturer Product Number (none) -> GRM155R61A106ME11D
- C22: Manufacturer (none) -> KEMET; Manufacturer Product Number (none) -> C0402C222J5RACTU
- C23: Manufacturer (none) -> KEMET; Manufacturer Product Number (none) -> C0603C102J5RACTU
- C3, C5: Manufacturer (none) -> KYOCERA AVX; Manufacturer Product Number (none) -> 0603YC105JAT2A
- C35, C36: footprint BowelProbe:Cap0.1uF -> BowelProbe:Cap1uF; Manufacturer (none) -> KYOCERA AVX; Manufacturer Product Number (none) -> 0603YC105JAT2A
- C37, C38: Manufacturer (none) -> KEMET; Manufacturer Product Number (none) -> C0603C180C5GACTU
- C4, C7: Manufacturer (none) -> Murata Electronics; Manufacturer Product Number (none) -> GRM21BR71C475KE51L
- C6: Manufacturer (none) -> Murata Electronics; Manufacturer Product Number (none) -> GJM1555C1H4R7BB01D
- D1: MANUFACTURER Diotec Semiconductor -> (none); Manufacturer (none) -> Diotec Semiconductor; Manufacturer Product Number (none) -> SDB160WS-AQ
- D2: renamed from U6; Manufacturer (none) -> Diodes Incorporated; Manufacturer Product Number (none) -> BAS116-7-F
- D3: renamed from CR1; Manufacturer (none) -> Toshiba Semiconductor and Storage; Manufacturer Product Number (none) -> CUS10S30,H3F
- D4: renamed from CR2; Manufacturer (none) -> Toshiba Semiconductor and Storage; Manufacturer Product Number (none) -> CUS10S30,H3F
- HS1: MANUFACTURER Same Sky -> (none); Manufacturer (none) -> Same Sky; Manufacturer Product Number (none) -> HSE-B20380-040H
- J1, J10, J11, J12, J13, J14, J15, J16, J17, J18, J19, J2, J20, J3, J4, J6, J7, J8, J9: now left out of the parts list
- J5: Manufacturer (none) -> Sullins Connector Solutions; Manufacturer Product Number (none) -> PPPC032LFBN-RC
- L1: MANUFACTURER Coilcraft -> (none); Manufacturer (none) -> Coilcraft; Manufacturer Product Number (none) -> LPD5030-472MRC
- L2: Manufacturer (none) -> TDK; Manufacturer Product Number (none) -> MLF1608E100JT000
- R1: Manufacturer (none) -> YAGEO; Manufacturer Product Number (none) -> RC0805FR-0771K5L
- R10: Manufacturer (none) -> Vishay Dale; Manufacturer Product Number (none) -> CRCW08051K00FKEA
- R12, R13, R14, R3: Manufacturer (none) -> YAGEO; Manufacturer Product Number (none) -> RC0603FR-0710KL
- R2: Manufacturer (none) -> YAGEO; Manufacturer Product Number (none) -> RC1206FR-071ML
- R4, R5: Manufacturer (none) -> YAGEO; Manufacturer Product Number (none) -> RC1206FR-076K8L
- R6: Manufacturer (none) -> YAGEO; Manufacturer Product Number (none) -> RC1206FR-0730KL
- R7: Manufacturer (none) -> YAGEO; Manufacturer Product Number (none) -> RC1206FR-071K8L
- R8: Manufacturer (none) -> Vishay Dale; Manufacturer Product Number (none) -> RCS0603100RFKEA
- R9: Manufacturer (none) -> YAGEO; Manufacturer Product Number (none) -> RC1206FR-07300KL
- U1: MANUFACTURER STMicroelectronics -> (none); Manufacturer (none) -> STMicroelectronics; Manufacturer Product Number (none) -> L7805CV
- U2: Manufacturer (none) -> Analog Devices Inc.; Manufacturer Product Number (none) -> LT8330IDDB#TRMPBF
- U3: Manufacturer (none) -> Analog Devices Inc.; Manufacturer Product Number (none) -> AD9833BRMZ
- U4: Manufacturer (none) -> Texas Instruments; Manufacturer Product Number (none) -> OPA2134UA/2K5
- U5: Manufacturer (none) -> Texas Instruments; Manufacturer Product Number (none) -> TL072ACDR
- U6: renamed from U7; Manufacturer (none) -> Microchip Technology; Manufacturer Product Number (none) -> MCP6002-E/MC
- U7: renamed from U8; Manufacturer (none) -> Microchip Technology; Manufacturer Product Number (none) -> ATMEGA328P-MUR
- XTAL1: Manufacturer (none) -> EPSON; Manufacturer Product Number (none) -> TSX-3225 16.0000MF09Z-AC3

Commit message: KiCad Updates
Added buffer after wave AD9833 sine generation and coupling capacitor (as simulated in LTspice) to address loading on filter stage. Added symbol, footprint, 3D model, and spice model in corresponding folders.

Updated BOM with this new part and updated PCB layout with buffer parts.
Parts:
- added C28: 10u, BowelProbe:Cap10uF, symbol Device:C_Small
- added C29: 0.1u, BowelProbe:Cap0.1uF, symbol Device:C_Small
- added R1: 1k, BowelProbe:Resistor1k, symbol Device:R_US
- added U5: Buffer, BowelProbe:Buffer, symbol BowelProbe:Buffer
- renumbered C36 to C17, C35 to C18, C37 to C19, C38 to C20, C39 to C21, C40 to C22, C17 to C23, C18 to C24, C19 to C25, C20 to C26, C21 to C27, C22 to C30, C23 to C31, C24 to C32, C25 to C33, C26 to C34, C27 to C35, C28 to C36, C29 to C37, C30 to C38, C31 to C39, C32 to C40, C33 to C41, C34 to C42, R6 to R10, R7 to R11, R8 to R12, R9 to R13, R10 to R14, R1 to R2, R2 to R3, R12 to R4, R13 to R5, R14 to R6, R3 to R7, R4 to R8, R5 to R9, U7 to U3, U3 to U4, U4 to U6, U5 to U7, U6 to U8
Connections:
- net +12V: now also R1.1; no longer C1.1, U1.1 (INPUT)
- net +5V: now also C28.1, C29.1, U5.5 (V+)
- net GND: now also C28.2, C29.2, U5.2 (V-)
- net Vsingen: now also U5.1 (+IN); no longer R8.1
- new net: C1.1, R1.2, U1.1 (INPUT)
- new net Vsinbuf: R8.1, U5.3 (-IN), U5.4 (OUT)
Other:
- note added: "Sine Generation & Buffer"
- note removed: "Sine Generation"
- moved on the sheet: C1, C2, D3, HS1, U1

Commit message: PCB Layout Progress
Initial rough layout of parts into corresponding sections. Next up is to formalize signal, power, and SPI flow as well as specific component placements.
Parts:
- added J21: Conn_01x08, BowelProbe:microSD, symbol Connector_Generic:Conn_01x08
- C10, C11, C12, C13, C14, C15, C16, C8, C9: value 10u -> 0.1u; footprint BowelProbe:Cap10uF -> BowelProbe:Cap0.1uF; Manufacturer Product Number GRM155R61A106ME11D -> GRM033C71C104KE14D
Connections:
- net A2 is gone; now on net A3: J17.1 (Pin_1)
- net A3: no longer J18.1 (Pin_1)
- net A4: now also J18.1 (Pin_1); no longer J19.1 (Pin_1)
- net A5: now also J19.1 (Pin_1); no longer J20.1 (Pin_1)
- net A6: now also J20.1 (Pin_1)
- net GND: now also U8.3 (VINA+), J21.1 (Pin_1), J21.4 (Pin_4), J21.5 (Pin_5), J21.6 (Pin_6), J21.7 (Pin_7), J21.8 (Pin_8)
- net at U8.1 (VOUTA): now also U8.2 (VINA-)
- no-connect marks 5 -> 4
Other:
- note added: "Stitching Capacitors"
- note removed: "Long Power Trace Decoupling"

Commit message: Schematic and Layout Updates
Added 47 ohm resistors to schematic to reduce ringing of SPI through ports and added corresponding info to BOM. Set PCB layout. May make a few more small tweaks.
Parts:
- removed J12, J13, J14, J15, J16, J20: Conn_01x01, BowelProbe:CT3149-0, symbol Connector_Generic:Conn_01x01
- added R15, R16, R17, R18: 47, BowelProbe:Resistor47, symbol Device:R_Small_US
- renumbered J17 to J12, J18 to J13, J19 to J14, J21 to J15
Connections:
- net GND: no longer J6.3 (Pin_3)
- net MISO: now also R15.2, R17.2; no longer J6.5 (Pin_5), U3.16 (PB4)
- net MOSI: now also R16.2; no longer U3.15 (PB3)
- net SCK: now also R18.1; no longer U3.17 (PB5)
- new net: R17.1, U3.16 (PB4)
- new net: R18.2, U3.17 (PB5)
- new net: J6.5 (Pin_5), R15.1
- new net: R16.1, U3.15 (PB3)
- no-connect marks 4 -> 11
Other:
- moved on the sheet: J10, J11, J12, J13, J14, J15, J7, J8, J9

Commit message: PCB Layout Plan Finalized
Added more stitching capacitors in schematic. Decided on final layout and added necessary vias. Added NPTH M3 mounting holes.
Parts:
- removed J10, J11: Conn_01x01, BowelProbe:CT3149-0, symbol Connector_Generic:Conn_01x01
- added C43, C44: 0.1u, BowelProbe:Cap0.1uF, symbol Device:C_Small
Connections:
- net D3 is gone; now on net CD: U3.1 (PD3)
- net D4 is gone; now on net nSS: U3.2 (PD4)
- net +5V: now also R5.1, R6.1, C43.1, C44.1; no longer R5.2, R6.2
- net CD: now also R5.2; no longer R6.1, U3.13 (PB1)
- net GND: now also C43.2, C44.2
- net nSS: now also R6.2; no longer R5.1, U3.14 (PB2)
- no-connect marks 11 -> 13
Other:
- moved on the sheet: J7, J8, J9, R5

Commit message: PCB Layout Routed
Schematic references adjusted and extra stitching capacitors removed. Layout added a few vias and fully routed.

Layout Finalization:
- Add ground pours on L1 and L4
- Add stitching vias
- Add edge stitching vias
- Review
Parts:
- removed C15, C16: 0.1u, BowelProbe:Cap0.1uF, symbol Device:C_Small
- renumbered C43 to C12, C12 to C13, C44 to C14, C13 to C15, C14 to C16, J14 to J10, J5 to J11, J3 to J12, J4 to J13, J6 to J3, J15 to J4, J7 to J5, J8 to J6, J9 to J7, J12 to J8, J13 to J9, R15 to R10, R7 to R11, R8 to R12, R9 to R13, R10 to R14, R11 to R15, R12 to R16, R13 to R17, R14 to R18, R16 to R7, R17 to R8, R18 to R9
Other:
- moved on the sheet: C16
